File: kicad_8bitLoveTape/LoveTape-2-2.kicad_pcb (KiCad board)
At the start: 2 copper layers, 66.9 x 63.4 mm, 13 parts, among them J1 audio out, SW3 On-Off, U1 ATTINY85-20PU

Commit message: fix some bad routings...
Parts:
- moved btn1 1.48 mm to (138.2, 114.1)
Connections:
- J1 pad 4: Net-(J1-Pad2) -> Net-(J1-Pad4)
- J1 pad 5: Net-(J1-Pad2) -> Net-(J1-Pad5)
- SW3 pad 3: (no net) -> Net-(SW3-Pad3)
- U1 pad 1: (no net) -> Net-(U1-Pad1)
Routing:
- net Net-(BT1-Pad2): track 67.3 -> 64.0 mm
- net Net-(J1-Pad2): track 35.0 -> 37.1 mm
- added copper zone on B.Cu, net GND
- added copper zone on B.Cu, net Net-(J1-Pad2)
Other:
- board text added: "+"
- board text added: "-"
- board text added: "8bit"
- board text added: "LovE tApE"
- board text removed: "8bit LovE"
- board text removed: "tapE"
